File: Hardware/OPI Hat/TPCastHat.kicad_sch (KiCad schematic)
At the start: 21 parts, among them J1 SOLDER_20AWG, J2 SOLDER_20AWG, J3 OPI Lite2 Header, J4 DCJack VID_RX_PWR, SW1 POWER_SW, U1 ADS1115IDGS, U2 INA219BxD, U3 TPS565208

Commit message: More changes to pcb design
Parts:
- added C4: 22µF, Capacitor_SMD:C_0805_2012Metric, symbol Device:C_Small
- C1: value 10uF -> 10µF; footprint (none) -> Capacitor_SMD:C_0805_2012Metric
- C2, C3: value 0.1uF -> 0.1µF; footprint (none) -> Capacitor_SMD:C_0805_2012Metric
- C5: renamed from C4; value 22uF -> 22µF; footprint (none) -> Capacitor_SMD:C_0805_2012Metric
- D1: footprint (none) -> _LocalParts:STPS30L30CG
- L1: value L_Small -> 3.3µH; footprint (none) -> Capacitor_SMD:C_0805_2012Metric
- R1: footprint (none) -> Resistor_SMD:R_1206_3216Metric
- R2, R3, R4, R5, R6: footprint (none) -> Resistor_SMD:R_0805_2012Metric
Connections:
- net +5V: now also C4.1
- net GND: now also C4.2
- net VBAT_1: now also D1.3 (K); no longer D1.1 (K)
- net VBAT_2: now also D1.1 (K); no longer D1.3 (K)
Other:
- moved on the sheet: C1, C2, C3, C5, D1, J1, J2, J3, J4, L1, R1, R2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
